Commit message: fix: update URDF parameters and mesh files for Gemini 345Lg

File: orbbec_description/urdf/gemini345Lg.urdf.xacro (robot description, xacro)
@@ -9,15 +9,15 @@
     <inertial>
       <origin
-        xyz="-0.0134366415045081 0.00104651333898482 -7.03343267068714E-05"
-        rpy="0 0 0" />
-      <mass
-        value="0.0215844638416589" />
-      <inertia
-        ixx="3.27367097133559E-05"
-        ixy="1.00838588052087E-08"
-        ixz="-1.4724694847835E-10"
-        iyy="3.2433989304705E-06"
+        xyz="-0.00892631661319327 -0.0411953623128534 -6.74554835164257E-05"
+        rpy="0 0 0" />
+      <mass
+        value="0.0225056393827557" />
+      <inertia
+        ixx="3.27548632771085E-05"
+        ixy="1.00838588052088E-08"
+        ixz="-1.47247229793385E-10"
+        iyy="3.25729646992983E-06"
         iyz="-1.75779219489013E-07"
-        izz="3.12774671483993E-05" />
+        izz="3.12913646878586E-05" />
     </inertial>
     <visual>
@@ -49,5 +49,5 @@
     <inertial>
       <origin
-        xyz="-0.0350120894657584 -0.00340477075942242 8.70441866524275E-05"
+        xyz="0.00893791053424158 -0.0334047707594224 0.0110870441866524"
         rpy="0 0 0" />
       <mass
@@ -56,7 +56,7 @@
         ixx="1.88009660853793E-05"
         ixy="-4.43021080342314E-07"
-        ixz="-2.91588301648928E-09"
+        ixz="-2.9158830164892E-09"
         iyy="2.53990333445075E-06"
-        iyz="-2.8372782100572E-08"
+        iyz="-2.83727821005721E-08"
         izz="1.75573510554478E-05" />
     </inertial>
@@ -89,5 +89,5 @@
     type="fixed">
     <origin
-      xyz="0 0 0"
+      xyz="-0.039695 -0.0139999995 -0.011"
       rpy="0 0 0" />
     <parent
@@ -102,14 +102,14 @@
     <inertial>
       <origin
-        xyz="-0.00294368828819506 5.00000006675716E-10 -5.94655220111843E-11"
+        xyz="-0.00294368828819507 4.99999992797928E-10 -5.94655219848769E-11"
         rpy="0 0 0" />
       <mass
         value="0.000921175541096741" />
       <inertia
-        ixx="1.81535637526191E-08"
-        ixy="-4.65942125450868E-25"
-        ixz="-2.81315054199892E-16"
+        ixx="1.81535637526192E-08"
+        ixy="-3.44693528328977E-25"
+        ixz="-2.81315054108964E-16"
         iyy="1.38975394593283E-08"
-        iyz="-1.13821267266512E-33"
+        iyz="-1.0298650842081E-33"
         izz="1.38975394593283E-08" />
     </inertial>
@@ -142,5 +142,5 @@
     type="fixed">
     <origin
-      xyz="-0.004255 0.044 0"
+      xyz="0.039695 0.0139999995 0.011"
       rpy="0 0 0" />
     <parent
@@ -155,15 +155,15 @@
     <inertial>
       <origin
-        xyz="-5.00000006675716E-10 5.94655220374918E-11 -0.00294368828819506"
-        rpy="0 0 0" />
-      <mass
-        value="0.000921175541096741" />
+        xyz="-5.00000006675716E-10 5.94655219568156E-11 -0.00294368828819506"
+        rpy="0 0 0" />
+      <mass
+        value="0.000921175541096742" />
       <inertia
         ixx="1.38975394593283E-08"
-        ixy="-1.13821267159089E-33"
-        ixz="4.65942125450868E-25"
+        ixy="-1.02986508493708E-33"
+        ixz="3.44693528328977E-25"
         iyy="1.38975394593283E-08"
         iyz="2.8131505422727E-16"
-        izz="1.81535637526191E-08" />
+        izz="1.81535637526192E-08" />
     </inertial>
     <visual>
@@ -196,5 +196,5 @@
     <origin
       xyz="0 0 0"
-      rpy="-1.5708 0 -1.5708" />
+      rpy="-1.5707963267949 0 -1.5707963267949" />
     <parent
       link="camera_infra1_frame" />
@@ -208,5 +208,5 @@
     <inertial>
       <origin
-        xyz="-0.00294368828819506 0 -5.5946552198084E-10"
+        xyz="-0.00294368828819506 0 -5.59465521922963E-10"
         rpy="0 0 0" />
       <mass
@@ -214,8 +214,8 @@
       <inertia
         ixx="1.81535637526192E-08"
-        ixy="-4.65942125450868E-25"
-        ixz="-2.8131505407876E-16"
+        ixy="-3.44693528328977E-25"
+        ixz="-2.81315054152356E-16"
         iyy="1.38975394593283E-08"
-        iyz="-1.13821267070129E-33"
+        iyz="-1.02986508510413E-33"
         izz="1.38975394593283E-08" />
     </inertial>
@@ -248,5 +248,5 @@
     type="fixed">
     <origin
-      xyz="-0.004255 -0.044 0"
+      xyz="0.039695 -0.074 0.0110000005"
       rpy="0 0 0" />
     <parent
@@ -261,5 +261,5 @@
     <inertial>
       <origin
-        xyz="0 5.59465522005393E-10 -0.00294368828819506"
+        xyz="0 5.59465521977332E-10 -0.00294368828819506"
         rpy="0 0 0" />
       <mass
@@ -267,8 +267,8 @@
       <inertia
         ixx="1.38975394593283E-08"
-        ixy="-1.13821267174195E-33"
-        ixz="4.65942125450868E-25"
+        ixy="-1.02986508413216E-33"
+        ixz="3.44693528328977E-25"
         iyy="1.38975394593283E-08"
-        iyz="2.81315054258919E-16"
+        iyz="2.8131505407876E-16"
         izz="1.81535637526192E-08" />
     </inertial>
@@ -302,5 +302,5 @@
     <origin
       xyz="0 0 0"
-      rpy="-1.5708 0 -1.5708" />
+      rpy="-1.5707963267949 0 -1.5707963267949" />
     <parent
       link="camera_infra2_frame" />
@@ -314,5 +314,5 @@
     <inertial>
       <origin
-        xyz="-0.00321027945431743 9.00165896683403E-11 5.37104609194339E-11"
+        xyz="-0.00321027945431743 9.00165896683403E-11 5.37104607625836E-11"
         rpy="0 0 0" />
       <mass
@@ -320,6 +320,6 @@
       <inertia
         ixx="2.6533618139805E-08"
-        ixy="-3.84539876551798E-16"
-        ixz="6.34689842906247E-16"
+        ixy="-3.84539876604891E-16"
+        ixz="6.34689842973081E-16"
         iyy="2.41480807907502E-08"
         iyz="-1.37568595195541E-14"
@@ -354,5 +354,5 @@
     type="fixed">
     <origin
-      xyz="-0.0045649 0.008 0"
+      xyz="0.0393851 -0.022 0.011"
       rpy="0 0 0" />
     <parent
@@ -367,5 +367,5 @@
     <inertial>
       <origin
-        xyz="-9.00165896683403E-11 -5.37104607204212E-11 -0.00321027945431743"
+        xyz="-9.00165896683403E-11 -5.37104609114104E-11 -0.00321027945431743"
         rpy="0 0 0" />
       <mass
@@ -374,7 +374,7 @@
         ixx="2.41480807907502E-08"
         ixy="-1.37568595195541E-14"
-        ixz="3.84539876614159E-16"
+        ixz="3.84539876573512E-16"
         iyy="2.41486930542313E-08"
-        iyz="-6.34689842868342E-16"
+        iyz="-6.34689842767368E-16"
         izz="2.6533618139805E-08" />
     </inertial>
@@ -408,5 +408,5 @@
     <origin
       xyz="0 0 0"
-      rpy="-1.5708 0 -1.5708" />
+      rpy="-1.5707963267949 0 -1.5707963267949" />
     <parent
       link="camera_color_frame" />
@@ -460,5 +460,5 @@
     type="fixed">
     <origin
-      xyz="-0.02955 0.019913 -0.0022324"
+      xyz="0.0144000000000001 -0.0100874 0.0087676"
       rpy="0 0 0" />
     <parent
@@ -473,5 +473,5 @@
     <inertial>
       <origin
-        xyz="-0.00294368828819506 5.00000006675716E-10 -5.94655220374918E-11"
+        xyz="-0.00294368828819507 4.99999992797928E-10 -5.9465521983123E-11"
         rpy="0 0 0" />
       <mass
@@ -479,8 +479,8 @@
       <inertia
         ixx="1.81535637526192E-08"
-        ixy="-4.65942125450868E-25"
-        ixz="-2.81315054239185E-16"
+        ixy="-3.44693528328977E-25"
+        ixz="-2.8131505413785E-16"
         iyy="1.38975394593283E-08"
-        iyz="-1.13821267214479E-33"
+        iyz="-1.02986508542306E-33"
         izz="1.38975394593283E-08" />
     </inertial>
@@ -513,5 +513,5 @@
     type="fixed">
     <origin
-      xyz="-0.004255 0.044 0"
+      xyz="0.039695 0.0139999995 0.011"
       rpy="0 0 0" />
     <parent

Commit message: Refactor code structure for improved readability and maintainability

File: orbbec_description/urdf/gemini345Lg.urdf.xacro (robot description, xacro)
@@ -6,5 +6,5 @@
     <xacro:property name="mesh_path" value="package://orbbec_description/meshes/gemini345Lg/" />
   <link
-    name="base_link">
+    name="camera_link">
     <inertial>
       <origin
@@ -27,5 +27,5 @@
       <geometry>
         <mesh
-          filename="${mesh_path}base_link.STL" />
+          filename="${mesh_path}camera_link.STL" />
       </geometry>
       <material
@@ -41,5 +41,5 @@
       <geometry>
         <mesh
-          filename="${mesh_path}base_link.STL" />
+          filename="${mesh_path}camera_link.STL" />
       </geometry>
     </collision>
@@ -92,5 +92,5 @@
       rpy="0 0 0" />
     <parent
-      link="base_link" />
+      link="camera_link" />
     <child
       link="camera_bottom_screw_frame" />
@@ -99,5 +99,5 @@
   </joint>
   <link
-    name="camera_infra1_frame">
+    name="camera_left_ir_frame">
     <inertial>
       <origin
@@ -120,5 +120,5 @@
       <geometry>
         <mesh
-          filename="${mesh_path}camera_infra1_frame.STL" />
+          filename="${mesh_path}camera_left_ir_frame.STL" />
       </geometry>
       <material
@@ -134,10 +134,10 @@
       <geometry>
         <mesh
-          filename="${mesh_path}camera_infra1_frame.STL" />
-      </geometry>
-    </collision>
-  </link>
-  <joint
-    name="camera_infra1_frame"
+          filename="${mesh_path}camera_left_ir_frame.STL" />
+      </geometry>
+    </collision>
+  </link>
+  <joint
+    name="camera_left_ir_frame"
     type="fixed">
     <origin
@@ -147,10 +147,10 @@
       link="camera_bottom_screw_frame" />
     <child
-      link="camera_infra1_frame" />
-    <axis
-      xyz="0 0 0" />
-  </joint>
-  <link
-    name="camera_infra1_optical_frame">
+      link="camera_left_ir_frame" />
+    <axis
+      xyz="0 0 0" />
+  </joint>
+  <link
+    name="camera_left_ir_optical_frame">
     <inertial>
       <origin
@@ -173,5 +173,5 @@
       <geometry>
         <mesh
-          filename="${mesh_path}camera_infra1_optical_frame.STL" />
+          filename="${mesh_path}camera_left_ir_optical_frame.STL" />
       </geometry>
       <material
@@ -187,10 +187,10 @@
       <geometry>
         <mesh
-          filename="${mesh_path}camera_infra1_optical_frame.STL" />
-      </geometry>
-    </collision>
-  </link>
-  <joint
-    name="camera_infra1_optical_frame"
+          filename="${mesh_path}camera_left_ir_optical_frame.STL" />
+      </geometry>
+    </collision>
+  </link>
+  <joint
+    name="camera_left_ir_optical_frame"
     type="fixed">
     <origin
@@ -198,12 +198,12 @@
       rpy="-1.5707963267949 0 -1.5707963267949" />
     <parent
-      link="camera_infra1_frame" />
-    <child
-      link="camera_infra1_optical_frame" />
-    <axis
-      xyz="0 0 0" />
-  </joint>
-  <link
-    name="camera_infra2_frame">
+      link="camera_left_ir_frame" />
+    <child
+      link="camera_left_ir_optical_frame" />
+    <axis
+      xyz="0 0 0" />
+  </joint>
+  <link
+    name="camera_right_ir_frame">
     <inertial>
       <origin
@@ -226,5 +226,5 @@
       <geometry>
         <mesh
-          filename="${mesh_path}camera_infra2_frame.STL" />
+          filename="${mesh_path}camera_right_ir_frame.STL" />
       </geometry>
       <material
@@ -240,10 +240,10 @@
       <geometry>
         <mesh
-          filename="${mesh_path}camera_infra2_frame.STL" />
-      </geometry>
-    </collision>
-  </link>
-  <joint
-    name="camera_infra2_frame"
+          filename="${mesh_path}camera_right_ir_frame.STL" />
+      </geometry>
+    </collision>
+  </link>
+  <joint
+    name="camera_right_ir_frame"
     type="fixed">
     <origin
@@ -253,10 +253,10 @@
       link="camera_bottom_screw_frame" />
     <child
-      link="camera_infra2_frame" />
-    <axis
-      xyz="0 0 0" />
-  </joint>
-  <link
-    name="camera_infra2_optical_frame">
+      link="camera_right_ir_frame" />
+    <axis
+      xyz="0 0 0" />
+  </joint>
+  <link
+    name="camera_right_ir_optical_frame">
     <inertial>
       <origin
@@ -279,5 +279,5 @@
       <geometry>
         <mesh
-          filename="${mesh_path}camera_infra2_optical_frame.STL" />
+          filename="${mesh_path}camera_right_ir_optical_frame.STL" />
       </geometry>
       <material
@@ -293,10 +293,10 @@
       <geometry>
         <mesh
-          filename="${mesh_path}camera_infra2_optical_frame.STL" />
-      </geometry>
-    </collision>
-  </link>
-  <joint
-    name="camera_infra2_optical_frame"
+          filename="${mesh_path}camera_right_ir_optical_frame.STL" />
+      </geometry>
+    </collision>
+  </link>
+  <joint
+    name="camera_right_ir_optical_frame"
     type="fixed">
     <origin
@@ -304,7 +304,7 @@
       rpy="-1.5707963267949 0 -1.5707963267949" />
     <parent
-      link="camera_infra2_frame" />
-    <child
-      link="camera_infra2_optical_frame" />
+      link="camera_right_ir_frame" />
+    <child
+      link="camera_right_ir_optical_frame" />
     <axis
       xyz="0 0 0" />

Commit message: fix: update joint configurations and link references in URDF for Gemini 345Lg

File: orbbec_description/urdf/gemini345Lg.urdf.xacro (robot description, xacro)
@@ -86,13 +86,13 @@
   </link>
   <joint
-    name="camera_bottom_screw_frame"
-    type="fixed">
-    <origin
-      xyz="-0.039695 -0.0139999995 -0.011"
+    name="camera_link_joint"
+    type="fixed">
+    <origin
+      xyz="0.039695 0.0139999995 0.011"
       rpy="0 0 0" />
     <parent
+      link="camera_bottom_screw_frame" />
+    <child
       link="camera_link" />
-    <child
-      link="camera_bottom_screw_frame" />
     <axis
       xyz="0 0 0" />
@@ -142,8 +142,8 @@
     type="fixed">
     <origin
-      xyz="0.039695 0.0139999995 0.011"
+      xyz="0 0 0"
       rpy="0 0 0" />
     <parent
-      link="camera_bottom_screw_frame" />
+      link="camera_depth_frame" />
     <child
       link="camera_left_ir_frame" />
@@ -248,8 +248,8 @@
     type="fixed">
     <origin
-      xyz="0.039695 -0.074 0.0110000005"
+      xyz="0 -0.088 0"
       rpy="0 0 0" />
     <parent
-      link="camera_bottom_screw_frame" />
+      link="camera_depth_frame" />
     <child
       link="camera_right_ir_frame" />
@@ -354,8 +354,8 @@
     type="fixed">
     <origin
-      xyz="0.0393851 -0.022 0.011"
+      xyz="-0.0003099 -0.036 0"
       rpy="0 0 0" />
     <parent
-      link="camera_bottom_screw_frame" />
+      link="camera_depth_frame" />
     <child
       link="camera_color_frame" />
@@ -460,8 +460,8 @@
     type="fixed">
     <origin
-      xyz="0.0144000000000001 -0.0100874 0.0087676"
+      xyz="-0.025295 -0.0240874 -0.0022324"
       rpy="0 0 0" />
     <parent
-      link="camera_bottom_screw_frame" />
+      link="camera_depth_frame" />
     <child
       link="camera_IMU_frame" />
@@ -513,8 +513,8 @@
     type="fixed">
     <origin
-      xyz="0.039695 0.0139999995 0.011"
+      xyz="0 0 0"
       rpy="0 0 0" />
     <parent
-      link="camera_bottom_screw_frame" />
+      link="camera_link" />
     <child
       link="camera_depth_frame" />
