Commit message: feat: add virtual root link and joint connection in URDF for Gemini 345Lg

File: orbbec_description/urdf/test_gemini345Lg.urdf.xacro (robot description, xacro)
@@ -5,3 +5,11 @@
 <robot name="gemini345Lg" xmlns:xacro="http://ros.org/wiki/xacro">
     <xacro:include filename="gemini345Lg.urdf.xacro"/>
+    <!-- Define a virtual root link -->
+  <link name="base_link"/>
+  <!-- Connect the virtual root to the actual base link -->
+  <joint name="base_link_to_camera_bottom_screw_frame" type="fixed">
+    <parent link="base_link"/>
+    <child link="camera_bottom_screw_frame"/>
+    <origin xyz="0 0 0" rpy="0 0 0"/>
+  </joint>
 </robot>
