Commit message: Rename Gemini URDF files consistently

File: orbbec_description/urdf/gemini_335_Lg.urdf.xacro (robot description, xacro)
@@ -4,5 +4,5 @@
      Commit Version: 1.6.0-4-g7f85cfe  Build Version: 1.6.7995.38578
      For more information, please see http://wiki.ros.org/sw_urdf_exporter -->
-<robot xmlns:xacro="http://ros.org/wiki/xacro" name="gemini335_336Lg">
+<robot xmlns:xacro="http://ros.org/wiki/xacro" name="gemini_335_Lg">
     <xacro:property name="mesh_path" value="package://orbbec_description/meshes/gemini335Lg/" />
     <link

File: orbbec_description/urdf/test_gemini_2.urdf.xacro (robot description, xacro)
@@ -3,6 +3,6 @@
      Commit Version: 1.6.0-4-g7f85cfe  Build Version: 1.6.7995.38578
      For more information, please see http://wiki.ros.org/sw_urdf_exporter -->
-<robot name="gemini335Le" xmlns:xacro="http://ros.org/wiki/xacro">
-    <xacro:include filename="gemini335Le.urdf.xacro"/>
+<robot name="gemini_2" xmlns:xacro="http://ros.org/wiki/xacro">
+    <xacro:include filename="gemini_2.urdf.xacro"/>
     <!-- Define a virtual root link -->
   <link name="base_link"/>
@@ -11,5 +11,5 @@
     <parent link="base_link"/>
     <child link="camera_link"/>
-    <origin xyz="0.034005 0.0475 0.014048" rpy="0 0 0"/>
+    <origin xyz="0.01491 0.025 0.0125" rpy="0 0 0"/>
   </joint>
 </robot>

File: orbbec_description/urdf/test_gemini_2_L.urdf.xacro (robot description, xacro)
@@ -3,6 +3,6 @@
      Commit Version: 1.6.0-4-g7f85cfe  Build Version: 1.6.7995.38578
      For more information, please see http://wiki.ros.org/sw_urdf_exporter -->
-<robot name="gemini2L" xmlns:xacro="http://ros.org/wiki/xacro">
-    <xacro:include filename="gemini2L.urdf.xacro"/>
+<robot name="gemini_2_L" xmlns:xacro="http://ros.org/wiki/xacro">
+    <xacro:include filename="gemini_2_L.urdf.xacro"/>
     <!-- Define a virtual root link -->
   <link name="base_link"/>

File: orbbec_description/urdf/test_gemini_335_L.urdf.xacro (robot description, xacro)
@@ -3,6 +3,6 @@
      Commit Version: 1.6.0-4-g7f85cfe  Build Version: 1.6.7995.38578
      For more information, please see http://wiki.ros.org/sw_urdf_exporter -->
-<robot name="gemini335Lg" xmlns:xacro="http://ros.org/wiki/xacro">
-    <xacro:include filename="gemini335Lg.urdf.xacro"/>
+<robot name="gemini_335_L" xmlns:xacro="http://ros.org/wiki/xacro">
+    <xacro:include filename="gemini_335_L_336_L.urdf.xacro"/>
     <!-- Define a virtual root link -->
   <link name="base_link"/>
@@ -11,5 +11,5 @@
     <parent link="base_link"/>
     <child link="camera_link"/>
-    <origin xyz="0.0117149999999995 0.0475 0.0143111800025738" rpy="0 0 0"/>
+    <origin xyz="0.011715 0.0475 0.014311" rpy="0 0 0"/>
   </joint>
 </robot>

File: orbbec_description/urdf/test_gemini_335_Le.urdf.xacro (robot description, xacro)
@@ -3,6 +3,6 @@
      Commit Version: 1.6.0-4-g7f85cfe  Build Version: 1.6.7995.38578
      For more information, please see http://wiki.ros.org/sw_urdf_exporter -->
-<robot name="gemini335L" xmlns:xacro="http://ros.org/wiki/xacro">
-    <xacro:include filename="gemini335L_336L.urdf.xacro"/>
+<robot name="gemini_335_Le" xmlns:xacro="http://ros.org/wiki/xacro">
+    <xacro:include filename="gemini_335_Le.urdf.xacro"/>
     <!-- Define a virtual root link -->
   <link name="base_link"/>
@@ -11,5 +11,5 @@
     <parent link="base_link"/>
     <child link="camera_link"/>
-    <origin xyz="0.011715 0.0475 0.014311" rpy="0 0 0"/>
+    <origin xyz="0.034005 0.0475 0.014048" rpy="0 0 0"/>
   </joint>
 </robot>

File: orbbec_description/urdf/test_gemini_335_Lg.urdf.xacro (robot description, xacro)
@@ -3,6 +3,6 @@
      Commit Version: 1.6.0-4-g7f85cfe  Build Version: 1.6.7995.38578
      For more information, please see http://wiki.ros.org/sw_urdf_exporter -->
-<robot name="gemini336L" xmlns:xacro="http://ros.org/wiki/xacro">
-    <xacro:include filename="gemini335L_336L.urdf.xacro"/>
+<robot name="gemini_335_Lg" xmlns:xacro="http://ros.org/wiki/xacro">
+    <xacro:include filename="gemini_335_Lg.urdf.xacro"/>
     <!-- Define a virtual root link -->
   <link name="base_link"/>
@@ -11,5 +11,5 @@
     <parent link="base_link"/>
     <child link="camera_link"/>
-    <origin xyz="0.011715 0.0475 0.014311" rpy="0 0 0"/>
+    <origin xyz="0.0117149999999995 0.0475 0.0143111800025738" rpy="0 0 0"/>
   </joint>
 </robot>

File: orbbec_description/urdf/test_gemini_336_L.urdf.xacro (robot description, xacro)
@@ -3,6 +3,6 @@
      Commit Version: 1.6.0-4-g7f85cfe  Build Version: 1.6.7995.38578
      For more information, please see http://wiki.ros.org/sw_urdf_exporter -->
-<robot name="gemini2" xmlns:xacro="http://ros.org/wiki/xacro">
-    <xacro:include filename="gemini2.urdf.xacro"/>
+<robot name="gemini_336_L" xmlns:xacro="http://ros.org/wiki/xacro">
+    <xacro:include filename="gemini_335_L_336_L.urdf.xacro"/>
     <!-- Define a virtual root link -->
   <link name="base_link"/>
@@ -11,5 +11,5 @@
     <parent link="base_link"/>
     <child link="camera_link"/>
-    <origin xyz="0.01491 0.025 0.0125" rpy="0 0 0"/>
+    <origin xyz="0.011715 0.0475 0.014311" rpy="0 0 0"/>
   </joint>
 </robot>
