Commit message: fix: update joint origins and remove redundant visual/collision elements in URDF for Gemini 305 and 309 models

File: orbbec_description/urdf/gemini305_g.urdf.xacro (robot description, xacro)
@@ -21,27 +21,4 @@
         izz="6.08547247005231E-06" />
     </inertial>
-    <visual>
-      <origin
-        xyz="0 0 0"
-        rpy="0 0 1.570796326794897" />
-      <geometry>
-        <mesh
-          filename="${mesh_path}base_link.STL" />
-      </geometry>
-      <material
-        name="">
-        <color
-          rgba="0.631372549019608 0.686274509803922 0.749019607843137 1" />
-      </material>
-    </visual>
-    <collision>
-      <origin
-        xyz="0 0 0"
-        rpy="0 0 1.570796326794897" />
-      <geometry>
-        <mesh
-          filename="${mesh_path}base_link.STL" />
-      </geometry>
-    </collision>
   </link>
   <link
@@ -64,8 +41,8 @@
       <origin
         xyz="0 0 0"
-        rpy="0 0 1.570796326794897" />
-      <geometry>
-        <mesh
-          filename="${mesh_path}camera_bottom_screw.STL" />
+        rpy="3.141592653589793 0 1.570796326794897" />
+      <geometry>
+        <mesh
+          filename="${mesh_path}base_link.STL" />
       </geometry>
       <material
@@ -78,8 +55,8 @@
       <origin
         xyz="0 0 0"
-        rpy="0 0 1.570796326794897" />
-      <geometry>
-        <mesh
-          filename="${mesh_path}camera_bottom_screw.STL" />
+        rpy="3.141592653589793 0 1.570796326794897" />
+      <geometry>
+        <mesh
+          filename="${mesh_path}base_link.STL" />
       </geometry>
     </collision>
@@ -142,5 +119,5 @@
     type="fixed">
     <origin
-      xyz="-0.00900395097915 0.008050000000001 -0.0209939609855011"
+      xyz="0.008050000000001 -0.00899604902085 0.0209939609855011"
       rpy="0 0 0" />
     <parent
@@ -195,5 +172,5 @@
     type="fixed">
     <origin
-      xyz="0.00899604902085 0.008050000000001 -0.0209939609855011"
+      xyz="0.008050000000001 0.00900395097915 0.0209939609855011"
       rpy="0 0 0" />
     <parent
@@ -220,27 +197,4 @@
         izz="6.96711715818641E-10" />
     </inertial>
-    <visual>
-      <origin
-        xyz="0 0 0"
-        rpy="0 0 1.570796326794897" />
-      <geometry>
-        <mesh
-          filename="${mesh_path}USB.STL" />
-      </geometry>
-      <material
-        name="">
-        <color
-          rgba="1 1 1 1" />
-      </material>
-    </visual>
-    <collision>
-      <origin
-        xyz="0 0 0"
-        rpy="0 0 1.570796326794897" />
-      <geometry>
-        <mesh
-          filename="${mesh_path}USB.STL" />
-      </geometry>
-    </collision>
   </link>
   <joint
@@ -248,5 +202,5 @@
     type="fixed">
     <origin
-      xyz="0.014696049020854 -0.00269500000000168 -0.0209939609854729"
+      xyz="-0.00269500000000168 -0.014696049020854 0.0209939609854729"
       rpy="0 0 0" />
     <parent
@@ -273,27 +227,4 @@
         izz="1.63868643158484E-06" />
     </inertial>
-    <visual>
-      <origin
-        xyz="0 0 0"
-        rpy="0 0 1.570796326794897" />
-      <geometry>
-        <mesh
-          filename="${mesh_path}camera_rear_screw_R.STL" />
-      </geometry>
-      <material
-        name="">
-        <color
-          rgba="0.874509803921569 0.945098039215686 1 1" />
-      </material>
-    </visual>
-    <collision>
-      <origin
-        xyz="0 0 0"
-        rpy="0 0 1.570796326794897" />
-      <geometry>
-        <mesh
-          filename="${mesh_path}camera_rear_screw_R.STL" />
-      </geometry>
-    </collision>
   </link>
   <joint
@@ -301,5 +232,5 @@
     type="fixed">
     <origin
-      xyz="-0.00679999999999827 -0.02379999999999 -0.0209900000000301"
+      xyz="-0.02379999999999 -0.00680000000000172 0.0209900000000301"
       rpy="0 0 0" />
     <parent
@@ -354,5 +285,5 @@
     type="fixed">
     <origin
-      xyz="0.00680000000000172 -0.02379999999999 -0.0209900000000301"
+      xyz="-0.02379999999999 0.00679999999999827 0.0209900000000301"
       rpy="0 0 0" />
     <parent
@@ -407,5 +338,5 @@
     type="fixed">
     <origin
-      xyz="0 -0.033409999999996 -0.020993960985498"
+      xyz="-0.033409999999996 0 0.020993960985498"
       rpy="0 0 0" />
     <parent

File: orbbec_description/urdf/gemini309_g.urdf.xacro (robot description, xacro)
@@ -21,27 +21,4 @@
         izz="4.83457340761002E-06" />
     </inertial>
-    <visual>
-      <origin
-        xyz="0 0 0"
-        rpy="0 0 1.570796326794897" />
-      <geometry>
-        <mesh
-          filename="${mesh_path}camera_bottom_screw.STL" />
-      </geometry>
-      <material
-        name="">
-        <color
-          rgba="0.631372549019608 0.686274509803922 0.749019607843137 1" />
-      </material>
-    </visual>
-    <collision>
-      <origin
-        xyz="0 0 0"
-        rpy="0 0 1.570796326794897" />
-      <geometry>
-        <mesh
-          filename="${mesh_path}camera_bottom_screw.STL" />
-      </geometry>
-    </collision>
   </link>
   <link
@@ -89,5 +66,5 @@
     type="fixed">
     <origin
-      xyz="-0.009003950979152 0.008050000000002 -0.0209939609855101"
+      xyz="0.008050000000002 -0.008996049020848 0.0209939609855101"
       rpy="0 0 0" />
     <parent
@@ -142,5 +119,5 @@
     type="fixed">
     <origin
-      xyz="0.008996049020848 0.008050000000002 -0.0209939609855101"
+      xyz="0.008050000000002 0.009003950979152 0.0209939609855101"
       rpy="0 0 0" />
     <parent
@@ -195,5 +172,5 @@
     type="fixed">
     <origin
-      xyz="0.014696049020852 -0.00269500000000068 -0.0209939609854819"
+      xyz="-0.00269500000000068 -0.014696049020852 0.0209939609854819"
       rpy="0 0 0" />
     <parent
@@ -220,27 +197,4 @@
         izz="1.63868643158484E-06" />
     </inertial>
-    <visual>
-      <origin
-        xyz="0 0 0"
-        rpy="0 0 1.570796326794897" />
-      <geometry>
-        <mesh
-          filename="${mesh_path}camera_rear_screw_R.STL" />
-      </geometry>
-      <material
-        name="">
-        <color
-          rgba="0.874509803921569 0.945098039215686 1 1" />
-      </material>
-    </visual>
-    <collision>
-      <origin
-        xyz="0 0 0"
-        rpy="0 0 1.570796326794897" />
-      <geometry>
-        <mesh
-          filename="${mesh_path}camera_rear_screw_R.STL" />
-      </geometry>
-    </collision>
   </link>
   <joint
@@ -248,5 +202,5 @@
     type="fixed">
     <origin
-      xyz="-0.00680000000000851 -0.0137999999999964 -0.0209900000000397"
+      xyz="-0.0137999999999964 -0.00679999999999149 0.0209900000000397"
       rpy="0 0 0" />
     <parent
@@ -273,27 +227,4 @@
         izz="1.63868643158484E-06" />
     </inertial>
-    <visual>
-      <origin
-        xyz="0 0 0"
-        rpy="0 0 1.570796326794897" />
-      <geometry>
-        <mesh
-          filename="${mesh_path}camera_rear_screw_L.STL" />
-      </geometry>
-      <material
-        name="">
-        <color
-          rgba="0.874509803921569 0.945098039215686 1 1" />
-      </material>
-    </visual>
-    <collision>
-      <origin
-        xyz="0 0 0"
-        rpy="0 0 1.570796326794897" />
-      <geometry>
-        <mesh
-          filename="${mesh_path}camera_rear_screw_L.STL" />
-      </geometry>
-    </collision>
   </link>
   <joint
@@ -301,5 +232,5 @@
     type="fixed">
     <origin
-      xyz="0.00679999999999149 -0.0137999999999964 -0.0209900000000397"
+      xyz="-0.0137999999999964 0.00680000000000851 0.0209900000000397"
       rpy="0 0 0" />
     <parent
@@ -329,5 +260,5 @@
       <origin
         xyz="0 0 0"
-        rpy="0 0 1.570796326794897" />
+        rpy="3.141592653589793 0 1.570796326794897" />
       <geometry>
         <mesh
@@ -354,5 +285,5 @@
     type="fixed">
     <origin
-      xyz="0 -0.0234099999999966 -0.0209939609855071"
+      xyz="-0.0234099999999966 0 0.0209939609855071"
       rpy="0 0 0" />
     <parent

Commit message: fix: remove camera rear screw links and joints from URDF for Gemini 305

File: orbbec_description/urdf/gemini305_g.urdf.xacro (robot description, xacro)
@@ -182,87 +182,4 @@
   </joint>
   <link
-    name="camera_rear_screw_R">
-    <inertial>
-      <origin
-        xyz="0.00694483634502586 -0.000403960805324607 -0.00046775323322587"
-        rpy="0 0 0" />
-      <mass
-        value="0.00885761204737663" />
-      <inertia
-        ixx="1.66869077460572E-06"
-        ixy="-2.55469491377221E-10"
-        ixz="7.6968875169436E-09"
-        iyy="3.1776766369675E-06"
-        iyz="-1.12550987680074E-09"
-        izz="1.63868643158484E-06" />
-    </inertial>
-  </link>
-  <joint
-    name="camera_rear_screw_R"
-    type="fixed">
-    <origin
-      xyz="-0.02379999999999 -0.00680000000000172 0.0209900000000301"
-      rpy="0 0 0" />
-    <parent
-      link="base_link" />
-    <child
-      link="camera_rear_screw_R" />
-    <axis
-      xyz="0 0 0" />
-  </joint>
-  <link
-    name="camera_rear_screw_L">
-    <inertial>
-      <origin
-        xyz="-0.00665516365497414 -0.000403960805324607 -0.00046775323322587"
-        rpy="0 0 0" />
-      <mass
-        value="0.00885761204737663" />
-      <inertia
-        ixx="1.66869077460572E-06"
-        ixy="-2.55469491377209E-10"
-        ixz="7.69688751694358E-09"
-        iyy="3.1776766369675E-06"
-        iyz="-1.12550987680075E-09"
-        izz="1.63868643158484E-06" />
-    </inertial>
-    <visual>
-      <origin
-        xyz="0 0 0"
-        rpy="0 0 1.570796326794897" />
-      <geometry>
-        <mesh
-          filename="${mesh_path}camera_rear_screw_L.STL" />
-      </geometry>
-      <material
-        name="">
-        <color
-          rgba="0.874509803921569 0.945098039215686 1 1" />
-      </material>
-    </visual>
-    <collision>
-      <origin
-        xyz="0 0 0"
-        rpy="0 0 1.570796326794897" />
-      <geometry>
-        <mesh
-          filename="${mesh_path}camera_rear_screw_L.STL" />
-      </geometry>
-    </collision>
-  </link>
-  <joint
-    name="camera_rear_screw_L"
-    type="fixed">
-    <origin
-      xyz="-0.02379999999999 0.00679999999999827 0.0209900000000301"
-      rpy="0 0 0" />
-    <parent
-      link="base_link" />
-    <child
-      link="camera_rear_screw_L" />
-    <axis
-      xyz="0 0 0" />
-  </joint>
-  <link
     name="FAKRA">
     <inertial>
