Commit message: fix: adjust joint origins and remove redundant visual/collision elements in URDF for Gemini 305

File: orbbec_description/urdf/gemini305.urdf.xacro (robot description, xacro)
@@ -21,27 +21,4 @@
         izz="3.76189543642479E-06" />
     </inertial>
-    <visual>
-      <origin
-        xyz="0 0 0"
-        rpy="0 0 1.570796326794897" />
-      <geometry>
-        <mesh
-          filename="${mesh_path}base_link.STL" />
-      </geometry>
-      <material
-        name="">
-        <color
-          rgba="1 1 0.945098039215686 1" />
-      </material>
-    </visual>
-    <collision>
-      <origin
-        xyz="0 0 0"
-        rpy="0 0 1.570796326794897" />
-      <geometry>
-        <mesh
-          filename="${mesh_path}base_link.STL" />
-      </geometry>
-    </collision>
   </link>
   <link
@@ -89,5 +66,5 @@
     type="fixed">
     <origin
-      xyz="-0.008999999999889 0.008126703388352 -0.0210000000000001"
+      xyz="0.008126703388352 0.008999999999889 0.0210000000000001"
       rpy="0 0 0" />
     <parent
@@ -142,5 +119,5 @@
     type="fixed">
     <origin
-      xyz="0.009000000000111 0.008126703388352 -0.0210000000000001"
+      xyz="0.008126703388352 -0.009000000000111 0.0210000000000001"
       rpy="0 0 0" />
     <parent
@@ -195,5 +172,5 @@
     type="fixed">
     <origin
-      xyz="0.014700000000115 -0.00261829661165068 -0.0209999999999719"
+      xyz="-0.00261829661165068 -0.014700000000115 0.0209999999999719"
       rpy="0 0 0" />
     <parent
@@ -223,5 +200,5 @@
       <origin
         xyz="0 0 0"
-        rpy="0 0 1.570796326794897" />
+        rpy="3.141592653589793 0 1.570796326794897" />
       <geometry>
         <mesh
@@ -248,5 +225,5 @@
     type="fixed">
     <origin
-      xyz="-0.00999680631556896 -0.01091969797964 -0.0209990315919259"
+      xyz="-0.01091969797964 0.00999680631556896 0.0209990315919259"
       rpy="0 0 0" />
     <parent
@@ -276,5 +253,5 @@
       <origin
         xyz="0 0 0"
-        rpy="0 0 1.570796326794897" />
+        rpy="3.141592653589793 0 1.570796326794897" />
       <geometry>
         <mesh
@@ -290,5 +267,5 @@
       <origin
         xyz="0 0 0"
-        rpy="0 0 1.570796326794897" />
+        rpy="3.141592653589793 0 1.570796326794897" />
       <geometry>
         <mesh
@@ -301,5 +278,5 @@
     type="fixed">
     <origin
-      xyz="0.0100031936844311 -0.01091969797964 -0.0209990315919259"
+      xyz="-0.01091969797964 -0.0100031936844311 0.0209990315919259"
       rpy="0 0 0" />
     <parent
@@ -329,5 +306,5 @@
       <origin
         xyz="0 0 0"
-        rpy="0 0 1.570796326794897" />
+        rpy="3.141592653589793 0 1.570796326794897" />
       <geometry>
         <mesh
@@ -343,5 +320,5 @@
       <origin
         xyz="0 0 0"
-        rpy="0 0 1.570796326794897" />
+        rpy="3.141592653589793 0 1.570796326794897" />
       <geometry>
         <mesh

Commit message: fix: correct joint origin coordinates for RGB and camera rear screw links in URDF for Gemini 305

File: orbbec_description/urdf/gemini305.urdf.xacro (robot description, xacro)
@@ -66,4 +66,57 @@
     type="fixed">
     <origin
+      xyz="0.008126703388352 -0.009000000000111 0.0210000000000001"
+      rpy="0 0 0" />
+    <parent
+      link="base_link" />
+    <child
+      link="RGB_R" />
+    <axis
+      xyz="0 0 0" />
+  </joint>
+  <link
+    name="RGB_L">
+    <inertial>
+      <origin
+        xyz="-0.00880445047118283 -0.00818012505851481 0.000610136627721265"
+        rpy="0 0 0" />
+      <mass
+        value="0.0195706749601595" />
+      <inertia
+        ixx="3.90938897723015E-06"
+        ixy="-1.54949883302202E-09"
+        ixz="2.45880849146858E-08"
+        iyy="6.7877667129966E-06"
+        iyz="-9.63634999610214E-09"
+        izz="3.76189543642479E-06" />
+    </inertial>
+    <visual>
+      <origin
+        xyz="0 0 0"
+        rpy="0 0 1.570796326794897" />
+      <geometry>
+        <mesh
+          filename="${mesh_path}RGB_L.STL" />
+      </geometry>
+      <material
+        name="">
+        <color
+          rgba="0.956862745098039 0.0470588235294118 0.874509803921569 1" />
+      </material>
+    </visual>
+    <collision>
+      <origin
+        xyz="0 0 0"
+        rpy="0 0 1.570796326794897" />
+      <geometry>
+        <mesh
+          filename="${mesh_path}RGB_L.STL" />
+      </geometry>
+    </collision>
+  </link>
+  <joint
+    name="RGB_L"
+    type="fixed">
+    <origin
       xyz="0.008126703388352 0.008999999999889 0.0210000000000001"
       rpy="0 0 0" />
@@ -71,19 +124,19 @@
       link="base_link" />
     <child
-      link="RGB_R" />
-    <axis
-      xyz="0 0 0" />
-  </joint>
-  <link
-    name="RGB_L">
-    <inertial>
-      <origin
-        xyz="-0.00880445047118283 -0.00818012505851481 0.000610136627721265"
-        rpy="0 0 0" />
-      <mass
-        value="0.0195706749601595" />
-      <inertia
-        ixx="3.90938897723015E-06"
-        ixy="-1.54949883302202E-09"
+      link="RGB_L" />
+    <axis
+      xyz="0 0 0" />
+  </joint>
+  <link
+    name="USB">
+    <inertial>
+      <origin
+        xyz="-0.0145044504711869 0.00256487494148787 0.000610136627693075"
+        rpy="0 0 0" />
+      <mass
+        value="0.0195706749601595" />
+      <inertia
+        ixx="3.90938897723015E-06"
+        ixy="-1.54949883302208E-09"
         ixz="2.45880849146858E-08"
         iyy="6.7877667129966E-06"
@@ -97,40 +150,40 @@
       <geometry>
         <mesh
-          filename="${mesh_path}RGB_L.STL" />
-      </geometry>
-      <material
-        name="">
-        <color
-          rgba="0.956862745098039 0.0470588235294118 0.874509803921569 1" />
-      </material>
-    </visual>
-    <collision>
-      <origin
-        xyz="0 0 0"
-        rpy="0 0 1.570796326794897" />
-      <geometry>
-        <mesh
-          filename="${mesh_path}RGB_L.STL" />
-      </geometry>
-    </collision>
-  </link>
-  <joint
-    name="RGB_L"
-    type="fixed">
-    <origin
-      xyz="0.008126703388352 -0.009000000000111 0.0210000000000001"
-      rpy="0 0 0" />
-    <parent
-      link="base_link" />
-    <child
-      link="RGB_L" />
-    <axis
-      xyz="0 0 0" />
-  </joint>
-  <link
-    name="USB">
-    <inertial>
-      <origin
-        xyz="-0.0145044504711869 0.00256487494148787 0.000610136627693075"
+          filename="${mesh_path}USB.STL" />
+      </geometry>
+      <material
+        name="">
+        <color
+          rgba="1 1 1 1" />
+      </material>
+    </visual>
+    <collision>
+      <origin
+        xyz="0 0 0"
+        rpy="0 0 1.570796326794897" />
+      <geometry>
+        <mesh
+          filename="${mesh_path}USB.STL" />
+      </geometry>
+    </collision>
+  </link>
+  <joint
+    name="USB"
+    type="fixed">
+    <origin
+      xyz="-0.00261829661165068 -0.014700000000115 0.0209999999999719"
+      rpy="0 0 0" />
+    <parent
+      link="base_link" />
+    <child
+      link="USB" />
+    <axis
+      xyz="0 0 0" />
+  </joint>
+  <link
+    name="camera_rear_screw_R">
+    <inertial>
+      <origin
+        xyz="0.0101923558444971 0.0108662763094772 0.000609168219647137"
         rpy="0 0 0" />
       <mass
@@ -141,57 +194,4 @@
         ixz="2.45880849146858E-08"
         iyy="6.7877667129966E-06"
-        iyz="-9.63634999610214E-09"
-        izz="3.76189543642479E-06" />
-    </inertial>
-    <visual>
-      <origin
-        xyz="0 0 0"
-        rpy="0 0 1.570796326794897" />
-      <geometry>
-        <mesh
-          filename="${mesh_path}USB.STL" />
-      </geometry>
-      <material
-        name="">
-        <color
-          rgba="1 1 1 1" />
-      </material>
-    </visual>
-    <collision>
-      <origin
-        xyz="0 0 0"
-        rpy="0 0 1.570796326794897" />
-      <geometry>
-        <mesh
-          filename="${mesh_path}USB.STL" />
-      </geometry>
-    </collision>
-  </link>
-  <joint
-    name="USB"
-    type="fixed">
-    <origin
-      xyz="-0.00261829661165068 -0.014700000000115 0.0209999999999719"
-      rpy="0 0 0" />
-    <parent
-      link="base_link" />
-    <child
-      link="USB" />
-    <axis
-      xyz="0 0 0" />
-  </joint>
-  <link
-    name="camera_rear_screw_R">
-    <inertial>
-      <origin
-        xyz="0.0101923558444971 0.0108662763094772 0.000609168219647137"
-        rpy="0 0 0" />
-      <mass
-        value="0.0195706749601595" />
-      <inertia
-        ixx="3.90938897723015E-06"
-        ixy="-1.54949883302208E-09"
-        ixz="2.45880849146858E-08"
-        iyy="6.7877667129966E-06"
         iyz="-9.63634999610213E-09"
         izz="3.76189543642479E-06" />
@@ -225,58 +225,58 @@
     type="fixed">
     <origin
+      xyz="-0.01091969797964 -0.0100031936844311 0.0209990315919259"
+      rpy="0 0 0" />
+    <parent
+      link="base_link" />
+    <child
+      link="camera_rear_screw_R" />
+    <axis
+      xyz="0 0 0" />
+  </joint>
+  <link
+    name="camera_rear_screw_L">
+    <inertial>
+      <origin
+        xyz="-0.00980764415550291 0.0108662763094772 0.000609168219647134"
+        rpy="0 0 0" />
+      <mass
+        value="0.0195706749601595" />
+      <inertia
+        ixx="3.90938897723015E-06"
+        ixy="-1.54949883302204E-09"
+        ixz="2.45880849146858E-08"
+        iyy="6.7877667129966E-06"
+        iyz="-9.63634999610211E-09"
+        izz="3.76189543642479E-06" />
+    </inertial>
+    <visual>
+      <origin
+        xyz="0 0 0"
+        rpy="3.141592653589793 0 1.570796326794897" />
+      <geometry>
+        <mesh
+          filename="${mesh_path}camera_rear_screw_L.STL" />
+      </geometry>
+      <material
+        name="">
+        <color
+          rgba="1 1 0.945098039215686 1" />
+      </material>
+    </visual>
+    <collision>
+      <origin
+        xyz="0 0 0"
+        rpy="3.141592653589793 0 1.570796326794897" />
+      <geometry>
+        <mesh
+          filename="${mesh_path}camera_rear_screw_L.STL" />
+      </geometry>
+    </collision>
+  </link>
+  <joint
+    name="camera_rear_screw_L"
+    type="fixed">
+    <origin
       xyz="-0.01091969797964 0.00999680631556896 0.0209990315919259"
-      rpy="0 0 0" />
-    <parent
-      link="base_link" />
-    <child
-      link="camera_rear_screw_R" />
-    <axis
-      xyz="0 0 0" />
-  </joint>
-  <link
-    name="camera_rear_screw_L">
-    <inertial>
-      <origin
-        xyz="-0.00980764415550291 0.0108662763094772 0.000609168219647134"
-        rpy="0 0 0" />
-      <mass
-        value="0.0195706749601595" />
-      <inertia
-        ixx="3.90938897723015E-06"
-        ixy="-1.54949883302204E-09"
-        ixz="2.45880849146858E-08"
-        iyy="6.7877667129966E-06"
-        iyz="-9.63634999610211E-09"
-        izz="3.76189543642479E-06" />
-    </inertial>
-    <visual>
-      <origin
-        xyz="0 0 0"
-        rpy="3.141592653589793 0 1.570796326794897" />
-      <geometry>
-        <mesh
-          filename="${mesh_path}camera_rear_screw_L.STL" />
-      </geometry>
-      <material
-        name="">
-        <color
-          rgba="1 1 0.945098039215686 1" />
-      </material>
-    </visual>
-    <collision>
-      <origin
-        xyz="0 0 0"
-        rpy="3.141592653589793 0 1.570796326794897" />
-      <geometry>
-        <mesh
-          filename="${mesh_path}camera_rear_screw_L.STL" />
-      </geometry>
-    </collision>
-  </link>
-  <joint
-    name="camera_rear_screw_L"
-    type="fixed">
-    <origin
-      xyz="-0.01091969797964 -0.0100031936844311 0.0209990315919259"
       rpy="0 0 0" />
     <parent

Commit message: fix: remove USB link and joint from URDF files for Gemini 305, 309 models

File: orbbec_description/urdf/gemini305.urdf.xacro (robot description, xacro)
@@ -129,57 +129,4 @@
   </joint>
   <link
-    name="USB">
-    <inertial>
-      <origin
-        xyz="-0.0145044504711869 0.00256487494148787 0.000610136627693075"
-        rpy="0 0 0" />
-      <mass
-        value="0.0195706749601595" />
-      <inertia
-        ixx="3.90938897723015E-06"
-        ixy="-1.54949883302208E-09"
-        ixz="2.45880849146858E-08"
-        iyy="6.7877667129966E-06"
-        iyz="-9.63634999610214E-09"
-        izz="3.76189543642479E-06" />
-    </inertial>
-    <visual>
-      <origin
-        xyz="0 0 0"
-        rpy="0 0 1.570796326794897" />
-      <geometry>
-        <mesh
-          filename="${mesh_path}USB.STL" />
-      </geometry>
-      <material
-        name="">
-        <color
-          rgba="1 1 1 1" />
-      </material>
-    </visual>
-    <collision>
-      <origin
-        xyz="0 0 0"
-        rpy="0 0 1.570796326794897" />
-      <geometry>
-        <mesh
-          filename="${mesh_path}USB.STL" />
-      </geometry>
-    </collision>
-  </link>
-  <joint
-    name="USB"
-    type="fixed">
-    <origin
-      xyz="-0.00261829661165068 -0.014700000000115 0.0209999999999719"
-      rpy="0 0 0" />
-    <parent
-      link="base_link" />
-    <child
-      link="USB" />
-    <axis
-      xyz="0 0 0" />
-  </joint>
-  <link
     name="camera_rear_screw_R">
     <inertial>

File: orbbec_description/urdf/gemini305_g.urdf.xacro (robot description, xacro)
@@ -182,34 +182,4 @@
   </joint>
   <link
-    name="USB">
-    <inertial>
-      <origin
-        xyz="-6.85782796221099E-05 -0.000107475646444261 -9.37341657112484E-06"
-        rpy="0 0 0" />
-      <mass
-        value="0.000124823132660932" />
-      <inertia
-        ixx="9.1168959979051E-10"
-        ixy="-1.5447084285369E-12"
-        ixz="-1.47259149967294E-12"
-        iyy="1.405009962927E-09"
-        iyz="-2.08275831584529E-14"
-        izz="6.96711715818641E-10" />
-    </inertial>
-  </link>
-  <joint
-    name="USB"
-    type="fixed">
-    <origin
-      xyz="-0.00269500000000168 -0.014696049020854 0.0209939609854729"
-      rpy="0 0 0" />
-    <parent
-      link="base_link" />
-    <child
-      link="USB" />
-    <axis
-      xyz="0 0 0" />
-  </joint>
-  <link
     name="camera_rear_screw_R">
     <inertial>

File: orbbec_description/urdf/gemini309_g.urdf.xacro (robot description, xacro)
@@ -129,26 +129,86 @@
   </joint>
   <link
-    name="USB">
-    <inertial>
-      <origin
-        xyz="-6.85782796221099E-05 -0.000107475646444262 -9.3734165711179E-06"
-        rpy="0 0 0" />
-      <mass
-        value="0.000124823132660932" />
-      <inertia
-        ixx="9.1168959979051E-10"
-        ixy="-1.54470842853689E-12"
-        ixz="-1.47259149967294E-12"
-        iyy="1.405009962927E-09"
-        iyz="-2.08275831583943E-14"
-        izz="6.96711715818641E-10" />
+    name="camera_rear_screw_R">
+    <inertial>
+      <origin
+        xyz="0.00694483634502586 -0.0004039608053246 -0.000467753233225888"
+        rpy="0 0 0" />
+      <mass
+        value="0.00885761204737661" />
+      <inertia
+        ixx="1.66869077460572E-06"
+        ixy="-2.55469491377294E-10"
+        ixz="7.69688751694532E-09"
+        iyy="3.1776766369675E-06"
+        iyz="-1.12550987680034E-09"
+        izz="1.63868643158484E-06" />
+    </inertial>
+  </link>
+  <joint
+    name="camera_rear_screw_R"
+    type="fixed">
+    <origin
+      xyz="-0.0137999999999964 -0.00679999999999149 0.0209900000000397"
+      rpy="0 0 0" />
+    <parent
+      link="camera_bottom_screw" />
+    <child
+      link="camera_rear_screw_R" />
+    <axis
+      xyz="0 0 0" />
+  </joint>
+  <link
+    name="camera_rear_screw_L">
+    <inertial>
+      <origin
+        xyz="-0.00665516365497414 -0.0004039608053246 -0.000467753233225888"
+        rpy="0 0 0" />
+      <mass
+        value="0.00885761204737661" />
+      <inertia
+        ixx="1.66869077460572E-06"
+        ixy="-2.55469491377279E-10"
+        ixz="7.69688751694532E-09"
+        iyy="3.1776766369675E-06"
+        iyz="-1.12550987680032E-09"
+        izz="1.63868643158484E-06" />
+    </inertial>
+  </link>
+  <joint
+    name="camera_rear_screw_L"
+    type="fixed">
+    <origin
+      xyz="-0.0137999999999964 0.00680000000000851 0.0209900000000397"
+      rpy="0 0 0" />
+    <parent
+      link="camera_bottom_screw" />
+    <child
+      link="camera_rear_screw_L" />
+    <axis
+      xyz="0 0 0" />
+  </joint>
+  <link
+    name="FAKRA">
+    <inertial>
+      <origin
+        xyz="0.000120342070480443 0.0189302142307225 0.000357727554186116"
+        rpy="0 0 0" />
+      <mass
+        value="0.0224266176030287" />
+      <inertia
+        ixx="4.90510990927456E-06"
+        ixy="-7.63213244507503E-10"
+        ixz="2.00360111638076E-08"
+        iyy="8.70411044641884E-06"
+        iyz="-2.68767067434135E-09"
+        izz="4.73094837296026E-06" />
     </inertial>
     <visual>
       <origin
         xyz="0 0 0"
-        rpy="0 0 1.570796326794897" />
-      <geometry>
-        <mesh
-          filename="${mesh_path}USB.STL" />
+        rpy="3.141592653589793 0 1.570796326794897" />
+      <geometry>
+        <mesh
+          filename="${mesh_path}FAKRA.STL" />
       </geometry>
       <material
@@ -164,122 +224,9 @@
       <geometry>
         <mesh
-          filename="${mesh_path}USB.STL" />
+          filename="${mesh_path}FAKRA.STL" />
       </geometry>
     </collision>
   </link>
   <joint
-    name="USB"
-    type="fixed">
-    <origin
-      xyz="-0.00269500000000068 -0.014696049020852 0.0209939609854819"
-      rpy="0 0 0" />
-    <parent
-      link="camera_bottom_screw" />
-    <child
-      link="USB" />
-    <axis
-      xyz="0 0 0" />
-  </joint>
-  <link
-    name="camera_rear_screw_R">
-    <inertial>
-      <origin
-        xyz="0.00694483634502586 -0.0004039608053246 -0.000467753233225888"
-        rpy="0 0 0" />
-      <mass
-        value="0.00885761204737661" />
-      <inertia
-        ixx="1.66869077460572E-06"
-        ixy="-2.55469491377294E-10"
-        ixz="7.69688751694532E-09"
-        iyy="3.1776766369675E-06"
-        iyz="-1.12550987680034E-09"
-        izz="1.63868643158484E-06" />
-    </inertial>
-  </link>
-  <joint
-    name="camera_rear_screw_R"
-    type="fixed">
-    <origin
-      xyz="-0.0137999999999964 -0.00679999999999149 0.0209900000000397"
-      rpy="0 0 0" />
-    <parent
-      link="camera_bottom_screw" />
-    <child
-      link="camera_rear_screw_R" />
-    <axis
-      xyz="0 0 0" />
-  </joint>
-  <link
-    name="camera_rear_screw_L">
-    <inertial>
-      <origin
-        xyz="-0.00665516365497414 -0.0004039608053246 -0.000467753233225888"
-        rpy="0 0 0" />
-      <mass
-        value="0.00885761204737661" />
-      <inertia
-        ixx="1.66869077460572E-06"
-        ixy="-2.55469491377279E-10"
-        ixz="7.69688751694532E-09"
-        iyy="3.1776766369675E-06"
-        iyz="-1.12550987680032E-09"
-        izz="1.63868643158484E-06" />
-    </inertial>
-  </link>
-  <joint
-    name="camera_rear_screw_L"
-    type="fixed">
-    <origin
-      xyz="-0.0137999999999964 0.00680000000000851 0.0209900000000397"
-      rpy="0 0 0" />
-    <parent
-      link="camera_bottom_screw" />
-    <child
-      link="camera_rear_screw_L" />
-    <axis
-      xyz="0 0 0" />
-  </joint>
-  <link
-    name="FAKRA">
-    <inertial>
-      <origin
-        xyz="0.000120342070480443 0.0189302142307225 0.000357727554186116"
-        rpy="0 0 0" />
-      <mass
-        value="0.0224266176030287" />
-      <inertia
-        ixx="4.90510990927456E-06"
-        ixy="-7.63213244507503E-10"
-        ixz="2.00360111638076E-08"
-        iyy="8.70411044641884E-06"
-        iyz="-2.68767067434135E-09"
-        izz="4.73094837296026E-06" />
-    </inertial>
-    <visual>
-      <origin
-        xyz="0 0 0"
-        rpy="3.141592653589793 0 1.570796326794897" />
-      <geometry>
-        <mesh
-          filename="${mesh_path}FAKRA.STL" />
-      </geometry>
-      <material
-        name="">
-        <color
-          rgba="1 1 1 1" />
-      </material>
-    </visual>
-    <collision>
-      <origin
-        xyz="0 0 0"
-        rpy="0 0 1.570796326794897" />
-      <geometry>
-        <mesh
-          filename="${mesh_path}FAKRA.STL" />
-      </geometry>
-    </collision>
-  </link>
-  <joint
     name="FAKRA"
     type="fixed">
