Commit message: fix: add camera joints and links in URDF for Gemini 305, 309 models

File: orbbec_description/urdf/gemini305.urdf.xacro (robot description, xacro)
@@ -6,22 +6,50 @@
   <xacro:property name="mesh_path" value="package://orbbec_description/meshes/gemini305/" />
   <link
-    name="base_link">
-    <inertial>
-      <origin
-        xyz="0.000195549528928161 -5.34216701628021E-05 -0.0203898633722788"
-        rpy="0 0 0" />
-      <mass
-        value="0.0195706749601595" />
-      <inertia
-        ixx="3.90938897723015E-06"
-        ixy="-1.54949883302207E-09"
-        ixz="2.45880849146858E-08"
-        iyy="6.7877667129966E-06"
-        iyz="-9.63634999610215E-09"
-        izz="3.76189543642479E-06" />
-    </inertial>
-  </link>
-  <link
-    name="RGB_R">
+    name="camera_link" />
+  <joint
+    name="camera_link"
+    type="fixed">
+    <origin
+      xyz="0.008126703388352 0.008999999999889 0.0210000000000001"
+      rpy="0 0 0" />
+    <parent
+      link="camera_bottom_screw" />
+    <child
+      link="camera_link" />
+    <axis
+      xyz="0 0 0" />
+  </joint>
+  <link
+    name="camera_left_color_optical_frame" />
+  <joint
+    name="camera_left_color_optical_frame"
+    type="fixed">
+    <origin
+      xyz="0 0 0"
+      rpy="-1.5707963267949 0 -1.5707963267949" />
+    <parent
+      link="camera_left_color_frame" />
+    <child
+      link="camera_left_color_optical_frame" />
+    <axis
+      xyz="0 0 0" />
+  </joint>
+  <link
+    name="camera_right_color_optical_frame" />
+  <joint
+    name="camera_right_color_optical_frame"
+    type="fixed">
+    <origin
+      xyz="0 0 0"
+      rpy="-1.5707963267949 0 -1.5707963267949" />
+    <parent
+      link="camera_right_color_frame" />
+    <child
+      link="camera_right_color_optical_frame" />
+    <axis
+      xyz="0 0 0" />
+  </joint>
+  <link
+    name="camera_right_color_frame">
     <inertial>
       <origin
@@ -63,18 +91,18 @@
   </link>
   <joint
-    name="RGB_R"
-    type="fixed">
-    <origin
-      xyz="0.008126703388352 -0.009000000000111 0.0210000000000001"
-      rpy="0 0 0" />
-    <parent
-      link="base_link" />
-    <child
-      link="RGB_R" />
-    <axis
-      xyz="0 0 0" />
-  </joint>
-  <link
-    name="RGB_L">
+    name="camera_right_color_frame"
+    type="fixed">
+    <origin
+      xyz="0 -0.018 0"
+      rpy="0 0 0" />
+    <parent
+      link="camera_left_color_frame" />
+    <child
+      link="camera_right_color_frame" />
+    <axis
+      xyz="0 0 0" />
+  </joint>
+  <link
+    name="camera_left_color_frame">
     <inertial>
       <origin
@@ -116,13 +144,13 @@
   </link>
   <joint
-    name="RGB_L"
-    type="fixed">
-    <origin
-      xyz="0.008126703388352 0.008999999999889 0.0210000000000001"
-      rpy="0 0 0" />
-    <parent
-      link="base_link" />
-    <child
-      link="RGB_L" />
+    name="camera_left_color_frame"
+    type="fixed">
+    <origin
+      xyz="0 0 0"
+      rpy="0 0 0" />
+    <parent
+      link="camera_link" />
+    <child
+      link="camera_left_color_frame" />
     <axis
       xyz="0 0 0" />
@@ -175,5 +203,5 @@
       rpy="0 0 0" />
     <parent
-      link="base_link" />
+      link="camera_bottom_screw" />
     <child
       link="camera_rear_screw_R" />
@@ -228,5 +256,5 @@
       rpy="0 0 0" />
     <parent
-      link="base_link" />
+      link="camera_bottom_screw" />
     <child
       link="camera_rear_screw_L" />
@@ -274,16 +302,3 @@
     </collision>
   </link>
-  <joint
-    name="camera_bottom_screw"
-    type="fixed">
-    <origin
-      xyz="0 0 0"
-      rpy="0 0 0" />
-    <parent
-      link="base_link" />
-    <child
-      link="camera_bottom_screw" />
-    <axis
-      xyz="0 0 0" />
-  </joint>
 </robot>

File: orbbec_description/urdf/gemini305_g.urdf.xacro (robot description, xacro)
@@ -6,20 +6,48 @@
   <xacro:property name="mesh_path" value="package://orbbec_description/meshes/gemini305_g/" />
   <link
-    name="base_link">
-    <inertial>
-      <origin
-        xyz="0.000149164489798296 -0.00906695064573543 -0.0207909592259398"
-        rpy="0 0 0" />
-      <mass
-        value="0.033546716795485" />
-      <inertia
-        ixx="6.61619826485559E-06"
-        ixy="-3.93814864956883E-09"
-        ixz="3.50980830227358E-08"
-        iyy="1.15876789717806E-05"
-        iyz="1.05717082804933E-08"
-        izz="6.08547247005231E-06" />
-    </inertial>
-  </link>
+    name="camera_link" />
+  <joint
+    name="camera_link"
+    type="fixed">
+    <origin
+      xyz="0.008050000000001 0.00900395097915 0.0209939609855011"
+      rpy="0 0 0" />
+    <parent
+      link="camera_bottom_screw" />
+    <child
+      link="camera_link" />
+    <axis
+      xyz="0 0 0" />
+  </joint>
+  <link
+    name="camera_left_color_optical_frame" />
+  <joint
+    name="camera_left_color_optical_frame"
+    type="fixed">
+    <origin
+      xyz="0 0 0"
+      rpy="-1.5707963267949 0 -1.5707963267949" />
+    <parent
+      link="camera_left_color_frame" />
+    <child
+      link="camera_left_color_optical_frame" />
+    <axis
+      xyz="0 0 0" />
+  </joint>
+  <link
+    name="camera_right_color_optical_frame" />
+  <joint
+    name="camera_right_color_optical_frame"
+    type="fixed">
+    <origin
+      xyz="0 0 0"
+      rpy="-1.5707963267949 0 -1.5707963267949" />
+    <parent
+      link="camera_right_color_frame" />
+    <child
+      link="camera_right_color_optical_frame" />
+    <axis
+      xyz="0 0 0" />
+  </joint>
   <link
     name="camera_bottom_screw">
@@ -61,20 +89,30 @@
       </geometry>
     </collision>
+    <visual>
+      <origin
+        xyz="-0.033409999999996 0 0.020993960985498"
+        rpy="0 0 1.570796326794897" />
+      <geometry>
+        <mesh
+          filename="${mesh_path}FAKRA.STL" />
+      </geometry>
+      <material
+        name="">
+        <color
+          rgba="1 1 1 1" />
+      </material>
+    </visual>
+    <collision>
+      <origin
+        xyz="-0.033409999999996 0 0.020993960985498"
+        rpy="0 0 1.570796326794897" />
+      <geometry>
+        <mesh
+          filename="${mesh_path}FAKRA.STL" />
+      </geometry>
+    </collision>
   </link>
-  <joint
-    name="camera_bottom_screw"
-    type="fixed">
-    <origin
-      xyz="0 0 0"
-      rpy="0 0 0" />
-    <parent
-      link="base_link" />
-    <child
-      link="camera_bottom_screw" />
-    <axis
-      xyz="0 0 0" />
-  </joint>
-  <link
-    name="RGB_R">
+  <link
+    name="camera_right_color_frame">
     <inertial>
       <origin
@@ -116,18 +154,18 @@
   </link>
   <joint
-    name="RGB_R"
-    type="fixed">
-    <origin
-      xyz="0.008050000000001 -0.00899604902085 0.0209939609855011"
+    name="camera_right_color_frame"
+    type="fixed">
+    <origin
+      xyz="0 -0.018 0"
       rpy="0 0 0" />
     <parent
-      link="base_link" />
-    <child
-      link="RGB_R" />
-    <axis
-      xyz="0 0 0" />
-  </joint>
-  <link
-    name="RGB_L">
+      link="camera_left_color_frame" />
+    <child
+      link="camera_right_color_frame" />
+    <axis
+      xyz="0 0 0" />
+  </joint>
+  <link
+    name="camera_left_color_frame">
     <inertial>
       <origin
@@ -169,66 +207,13 @@
   </link>
   <joint
-    name="RGB_L"
-    type="fixed">
-    <origin
-      xyz="0.008050000000001 0.00900395097915 0.0209939609855011"
+    name="camera_left_color_frame"
+    type="fixed">
+    <origin
+      xyz="0 0 0"
       rpy="0 0 0" />
     <parent
-      link="base_link" />
-    <child
-      link="RGB_L" />
-    <axis
-      xyz="0 0 0" />
-  </joint>
-  <link
-    name="FAKRA">
-    <inertial>
-      <origin
-        xyz="-2.19014445062421E-07 0.0027197100224461 -0.00011127645937509"
-        rpy="0 0 0" />
-      <mass
-        value="0.000751156783355389" />
-      <inertia
-        ixx="1.51891738860674E-08"
-        ixy="4.67248857458133E-13"
-        ixz="-3.5218905561991E-13"
-        iyy="1.40267326812145E-08"
-        iyz="-2.75286777175686E-10"
-        izz="1.86427254797844E-08" />
-    </inertial>
-    <visual>
-      <origin
-        xyz="0 0 0"
-        rpy="0 0 1.570796326794897" />
-      <geometry>
-        <mesh
-          filename="${mesh_path}FAKRA.STL" />
-      </geometry>
-      <material
-        name="">
-        <color
-          rgba="1 1 1 1" />
-      </material>
-    </visual>
-    <collision>
-      <origin
-        xyz="0 0 0"
-        rpy="0 0 1.570796326794897" />
-      <geometry>
-        <mesh
-          filename="${mesh_path}FAKRA.STL" />
-      </geometry>
-    </collision>
-  </link>
-  <joint
-    name="FAKRA"
-    type="fixed">
-    <origin
-      xyz="-0.033409999999996 0 0.020993960985498"
-      rpy="0 0 0" />
-    <parent
-      link="base_link" />
-    <child
-      link="FAKRA" />
+      link="camera_link" />
+    <child
+      link="camera_left_color_frame" />
     <axis
       xyz="0 0 0" />

File: orbbec_description/urdf/gemini309_g.urdf.xacro (robot description, xacro)
@@ -5,4 +5,49 @@
 <robot xmlns:xacro="http://ros.org/wiki/xacro" name="gemini309_g">
   <xacro:property name="mesh_path" value="package://orbbec_description/meshes/gemini309_g/" />
+  <link
+    name="camera_link" />
+  <joint
+    name="camera_link"
+    type="fixed">
+    <origin
+      xyz="0.008050000000002 0.009003950979152 0.0209939609855101"
+      rpy="0 0 0" />
+    <parent
+      link="camera_bottom_screw" />
+    <child
+      link="camera_link" />
+    <axis
+      xyz="0 0 0" />
+  </joint>
+  <link
+    name="camera_left_color_optical_frame" />
+  <joint
+    name="camera_left_color_optical_frame"
+    type="fixed">
+    <origin
+      xyz="0 0 0"
+      rpy="-1.5707963267949 0 -1.5707963267949" />
+    <parent
+      link="camera_left_color_frame" />
+    <child
+      link="camera_left_color_optical_frame" />
+    <axis
+      xyz="0 0 0" />
+  </joint>
+  <link
+    name="camera_right_color_optical_frame" />
+  <joint
+    name="camera_right_color_optical_frame"
+    type="fixed">
+    <origin
+      xyz="0 0 0"
+      rpy="-1.5707963267949 0 -1.5707963267949" />
+    <parent
+      link="camera_right_color_frame" />
+    <child
+      link="camera_right_color_optical_frame" />
+    <axis
+      xyz="0 0 0" />
+  </joint>
   <link
     name="camera_bottom_screw">
@@ -21,7 +66,30 @@
         izz="4.83457340761002E-06" />
     </inertial>
+    <visual>
+      <origin
+        xyz="-0.0234099999999966 0 0.0209939609855071"
+        rpy="3.141592653589793 0 1.570796326794897" />
+      <geometry>
+        <mesh
+          filename="${mesh_path}FAKRA.STL" />
+      </geometry>
+      <material
+        name="">
+        <color
+          rgba="1 1 1 1" />
+      </material>
+    </visual>
+    <collision>
+      <origin
+        xyz="-0.0234099999999966 0 0.0209939609855071"
+        rpy="3.141592653589793 0 1.570796326794897" />
+      <geometry>
+        <mesh
+          filename="${mesh_path}FAKRA.STL" />
+      </geometry>
+    </collision>
   </link>
   <link
-    name="RGB_R">
+    name="camera_right_color_frame">
     <inertial>
       <origin
@@ -63,18 +131,18 @@
   </link>
   <joint
-    name="RGB_R"
+    name="camera_right_color_frame"
     type="fixed">
     <origin
-      xyz="0.008050000000002 -0.008996049020848 0.0209939609855101"
+      xyz="0 -0.018 0"
       rpy="0 0 0" />
     <parent
-      link="camera_bottom_screw" />
+      link="camera_left_color_frame" />
     <child
-      link="RGB_R" />
+      link="camera_right_color_frame" />
     <axis
       xyz="0 0 0" />
   </joint>
   <link
-    name="RGB_L">
+    name="camera_left_color_frame">
     <inertial>
       <origin
@@ -116,126 +184,13 @@
   </link>
   <joint
-    name="RGB_L"
+    name="camera_left_color_frame"
     type="fixed">
     <origin
-      xyz="0.008050000000002 0.009003950979152 0.0209939609855101"
+      xyz="0 0 0"
       rpy="0 0 0" />
     <parent
-      link="camera_bottom_screw" />
+      link="camera_link" />
     <child
-      link="RGB_L" />
-    <axis
-      xyz="0 0 0" />
-  </joint>
-  <link
-    name="camera_rear_screw_R">
-    <inertial>
-      <origin
-        xyz="0.00694483634502586 -0.0004039608053246 -0.000467753233225888"
-        rpy="0 0 0" />
-      <mass
-        value="0.00885761204737661" />
-      <inertia
-        ixx="1.66869077460572E-06"
-        ixy="-2.55469491377294E-10"
-        ixz="7.69688751694532E-09"
-        iyy="3.1776766369675E-06"
-        iyz="-1.12550987680034E-09"
-        izz="1.63868643158484E-06" />
-    </inertial>
-  </link>
-  <joint
-    name="camera_rear_screw_R"
-    type="fixed">
-    <origin
-      xyz="-0.0137999999999964 -0.00679999999999149 0.0209900000000397"
-      rpy="0 0 0" />
-    <parent
-      link="camera_bottom_screw" />
-    <child
-      link="camera_rear_screw_R" />
-    <axis
-      xyz="0 0 0" />
-  </joint>
-  <link
-    name="camera_rear_screw_L">
-    <inertial>
-      <origin
-        xyz="-0.00665516365497414 -0.0004039608053246 -0.000467753233225888"
-        rpy="0 0 0" />
-      <mass
-        value="0.00885761204737661" />
-      <inertia
-        ixx="1.66869077460572E-06"
-        ixy="-2.55469491377279E-10"
-        ixz="7.69688751694532E-09"
-        iyy="3.1776766369675E-06"
-        iyz="-1.12550987680032E-09"
-        izz="1.63868643158484E-06" />
-    </inertial>
-  </link>
-  <joint
-    name="camera_rear_screw_L"
-    type="fixed">
-    <origin
-      xyz="-0.0137999999999964 0.00680000000000851 0.0209900000000397"
-      rpy="0 0 0" />
-    <parent
-      link="camera_bottom_screw" />
-    <child
-      link="camera_rear_screw_L" />
-    <axis
-      xyz="0 0 0" />
-  </joint>
-  <link
-    name="FAKRA">
-    <inertial>
-      <origin
-        xyz="0.000120342070480443 0.0189302142307225 0.000357727554186116"
-        rpy="0 0 0" />
-      <mass
-        value="0.0224266176030287" />
-      <inertia
-        ixx="4.90510990927456E-06"
-        ixy="-7.63213244507503E-10"
-        ixz="2.00360111638076E-08"
-        iyy="8.70411044641884E-06"
-        iyz="-2.68767067434135E-09"
-        izz="4.73094837296026E-06" />
-    </inertial>
-    <visual>
-      <origin
-        xyz="0 0 0"
-        rpy="3.141592653589793 0 1.570796326794897" />
-      <geometry>
-        <mesh
-          filename="${mesh_path}FAKRA.STL" />
-      </geometry>
-      <material
-        name="">
-        <color
-          rgba="1 1 1 1" />
-      </material>
-    </visual>
-    <collision>
-      <origin
-        xyz="0 0 0"
-        rpy="0 0 1.570796326794897" />
-      <geometry>
-        <mesh
-          filename="${mesh_path}FAKRA.STL" />
-      </geometry>
-    </collision>
-  </link>
-  <joint
-    name="FAKRA"
-    type="fixed">
-    <origin
-      xyz="-0.0234099999999966 0 0.0209939609855071"
-      rpy="0 0 0" />
-    <parent
-      link="camera_bottom_screw" />
-    <child
-      link="FAKRA" />
+      link="camera_left_color_frame" />
     <axis
       xyz="0 0 0" />
